Commit message: URDF Modified and Specific Tags Added

File: src/lid_description/models/ebot/ebot_description.xacro (robot description, xacro)
@@ -271,5 +271,5 @@
   <joint name="rplidar_joint" type="fixed">
     <axis xyz="0 1 0" />
-    <origin xyz="0.255540836099039 0 0.18"
+    <origin xyz="0.1 0.0 0.25"
       rpy="0 0 0.00679706827344463" />
     <parent link="base_link" />
@@ -619,5 +619,5 @@
   </joint>
   <!-- Camera link -->
-    <link name="camera_link">
+    <!-- <link name="camera_link">
       <collision>
         <origin xyz="0 0 0" rpy="0 0 0" />
@@ -637,7 +637,7 @@
         <inertia ixx="0" ixy="0" ixz="0" iyy="0" iyz="0" izz="0" />
       </inertial>
-    </link>
+    </link> -->
     <!-- Joint to parent -->
-    <joint name="camera_joint" type="fixed">
+    <!-- <joint name="camera_joint" type="fixed">
       <parent link="base_link" />
       <child link="camera_link" />
@@ -655,4 +655,4 @@
         <inertia ixx="1e-6" ixy="0" ixz="0" iyy="1e-6" iyz="0" izz="1e-6" />
       </inertial>
-    </link>
+    </link> -->
 </robot>
